Commit message: urdf finished

File: install/jetbot_ros/share/jetbot_ros/urdf/jetbot.urdf (robot description, URDF)
Before this commit: robot jetbot, 12 links, 11 joints
Links:
- removed link left_wheel_link
- removed link right_wheel_link
- added link left_wheel, mass 0.1; collision cylinder length=0.025 radius=0.0325; visual cylinder length=0.025 radius=0.0325
- added link right_wheel, mass 0.1; collision cylinder length=0.025 radius=0.0325; visual cylinder length=0.025 radius=0.0325
Joints:
- joint left_wheel_joint: child left_wheel_link -> left_wheel; limit effort=1000 velocity=1000 -> (none); origin xyz=0.05 0.0875 -0.0025 rpy=0 0 0 -> xyz=0.05 0.0875 0 rpy=0 0 0
- joint right_wheel_joint: child right_wheel_link -> right_wheel; limit effort=1000 velocity=1000 -> (none); origin xyz=0.05 -0.0875 -0.0025 rpy=0 0 0 -> xyz=0.05 -0.0875 0 rpy=0 0 0

File: install/jetbot_ros/share/jetbot_ros/urdf/jetbot.urdf.xacro (robot description, xacro)
@@ -2,4 +2,9 @@
 <robot name="jetbot" xmlns:xacro="http://www.ros.org/wiki/xacro">
 <!-- 尺寸定義 -->
+<!-- 參數定義 -->
+<xacro:property name="wheel_radius" value="0.0325"/>  <!-- 對應 wheel_link_radius -->
+<xacro:property name="wheel_thickness" value="0.025"/>  <!-- 對應 wheel_link_length -->
+<xacro:property name="wheel_distance" value="0.175"/>  <!-- 左右輪距 = 2 × 0.0875 -->
+<xacro:property name="wheel_x_offset" value="0.05"/>  <!-- 輪子前後位置 -->
 <xacro:property name="body_link_x_dim" value="0.20"/>
 <xacro:property name="body_link_y_dim" value="0.15"/>
@@ -8,5 +13,5 @@
 <xacro:property name="wheel_link_length" value="0.025"/>
 <xacro:property name="wheel_link_z_location" value="${-body_link_z_dim/2}"/>
-<xacro:property name="caster_link_radius" value="0.01"/>
+<xacro:property name="caster_link_radius" value="0.04"/>
 <xacro:property name="caster_link_z_location" value="${-body_link_z_dim/2-wheel_link_radius+caster_link_radius}"/>
 <xacro:property name="camera_radius" value="0.0025"/>
@@ -93,54 +98,67 @@
 </joint>
 <link name="base_link"/>
-<!-- 左輪：X=+0.05, Y=+0.0875 -->
+<!-- 左輪 -->
+<link name="left_wheel">
+    <visual>
+        <geometry>
+            <cylinder radius="${wheel_radius}" length="${wheel_thickness}"/>
+        </geometry>
+        <origin xyz="0 0 0" rpy="1.5708 0 0"/>  <!-- link 內設為 0 -->
+        <material name="black">
+            <color rgba="0.1 0.1 0.1 1.0"/>
+        </material>
+    </visual>
+    <collision>
+        <geometry>
+            <cylinder radius="${wheel_radius}" length="${wheel_thickness}"/>
+        </geometry>
+        <origin xyz="0 0 0" rpy="1.5708 0 0"/>  <!-- link 內設為 0 -->
+    </collision>
+    <inertial>
+        <mass value="0.1"/>
+        <origin xyz="0 0 0" rpy="0 0 0"/>
+        <inertia ixx="0.0001" ixy="0.0" ixz="0.0"
+                 iyy="0.0001" iyz="0.0"
+                 izz="0.0001"/>
+    </inertial>
+</link>
+<!-- 右輪 -->
+<link name="right_wheel">
+    <visual>
+        <geometry>
+            <cylinder radius="${wheel_radius}" length="${wheel_thickness}"/>
+        </geometry>
+        <origin xyz="0 0 0" rpy="1.5708 0 0"/>  <!-- link 內設為 0 -->
+        <material name="black"/>
+    </visual>
+    <collision>
+        <geometry>
+            <cylinder radius="${wheel_radius}" length="${wheel_thickness}"/>
+        </geometry>
+        <origin xyz="0 0 0" rpy="1.5708 0 0"/>  <!-- link 內設為 0 -->
+    </collision>
+    <inertial>
+        <mass value="0.1"/>
+        <origin xyz="0 0 0" rpy="0 0 0"/>
+        <inertia ixx="0.0001" ixy="0.0" ixz="0.0"
+                 iyy="0.0001" iyz="0.0"
+                 izz="0.0001"/>
+    </inertial>
+</link>
+<!-- 輪子關節 - 用你喜歡的格式 -->
 <joint name="left_wheel_joint" type="continuous">
     <parent link="body_link"/>
-    <child link="left_wheel_link"/>
-    <origin xyz="0.05 0.0875 ${wheel_link_z_location}" rpy="0 0 0"/>
+    <child link="left_wheel"/>
+    <origin xyz="${wheel_x_offset} ${wheel_distance/2} 0" rpy="0 0 0"/>
+    <!-- X=0.05, Y=0.0875, Z=0 -->
     <axis xyz="0 1 0"/>
-    <limit effort="1000" velocity="1000"/>
-    <dynamics damping="1.0" friction="1.0"/>
-</joint>
-<link name="left_wheel_link">
-    <visual>
-        <origin rpy="1.5708 0 0" xyz="0 0 0"/>
-        <geometry>
-            <cylinder length="${wheel_link_length}" radius="${wheel_link_radius}"/>
-        </geometry>
-        <material name="black"/>
-    </visual>
-    <collision>
-        <origin rpy="1.5708 0 0" xyz="0 0 0"/>
-        <geometry>
-            <cylinder length="${wheel_link_length}" radius="${wheel_link_radius}"/>
-        </geometry>
-    </collision>
-    <xacro:inertia_wheel/>
-</link>
-<!-- 右輪：X=+0.05, Y=-0.0875 -->
+</joint>
 <joint name="right_wheel_joint" type="continuous">
     <parent link="body_link"/>
-    <child link="right_wheel_link"/>
-    <origin xyz="0.05 -0.0875 ${wheel_link_z_location}" rpy="0 0 0"/>
+    <child link="right_wheel"/>
+    <origin xyz="${wheel_x_offset} ${-wheel_distance/2} 0" rpy="0 0 0"/>
+    <!-- X=0.05, Y=-0.0875, Z=0 -->
     <axis xyz="0 1 0"/>
-    <limit effort="1000" velocity="1000"/>
-    <dynamics damping="1.0" friction="1.0"/>
-</joint>
-<link name="right_wheel_link">
-    <visual>
-        <origin rpy="1.5708 0 0" xyz="0 0 0"/>
-        <geometry>
-            <cylinder length="${wheel_link_length}" radius="${wheel_link_radius}"/>
-        </geometry>
-        <material name="black"/>
-    </visual>
-    <collision>
-        <origin rpy="1.5708 0 0" xyz="0 0 0"/>
-        <geometry>
-            <cylinder length="${wheel_link_length}" radius="${wheel_link_radius}"/>
-        </geometry>
-    </collision>
-    <xacro:inertia_wheel/>
-</link>
+</joint>ㄋ
 <joint name="caster_joint" type="fixed">
     <parent link="body_link"/>

Commit message: 點雲part7

File: install/jetbot_ros/share/jetbot_ros/urdf/jetbot.urdf (robot description, URDF)
Before this commit: robot jetbot, 12 links, 11 joints
Links:
- link caster_link: mass 0.0041887902000000005 -> 0.26808257280000003; geometry collision sphere radius=0.04; visual sphere radius=0.04
- link left_wheel: mass 0.1 -> 0.08295768091406253
- link right_wheel: mass 0.1 -> 0.08295768091406253
Joints:
- joint caster_joint: origin xyz=-0.08 0 -0.025 rpy=0 0 0 -> xyz=-0.08 0 0.0049999999999999975 rpy=0 0 0
- joint left_wheel_joint: origin xyz=0.05 0.0875 0 rpy=0 0 0 -> xyz=0.05 0.09999999999999999 -0.0025 rpy=0 0 0
- joint right_wheel_joint: origin xyz=0.05 -0.0875 0 rpy=0 0 0 -> xyz=0.05 -0.09999999999999999 -0.0025 rpy=0 0 0

File: install/jetbot_ros/share/jetbot_ros/urdf/jetbot.urdf.xacro (robot description, xacro)
@@ -1,10 +1,8 @@
 <?xml version="1.0"?>
 <robot name="jetbot" xmlns:xacro="http://www.ros.org/wiki/xacro">
-<!-- 尺寸定義 -->
-<!-- 參數定義 -->
-<xacro:property name="wheel_radius" value="0.0325"/>  <!-- 對應 wheel_link_radius -->
-<xacro:property name="wheel_thickness" value="0.025"/>  <!-- 對應 wheel_link_length -->
-<xacro:property name="wheel_distance" value="0.175"/>  <!-- 左右輪距 = 2 × 0.0875 -->
-<xacro:property name="wheel_x_offset" value="0.05"/>  <!-- 輪子前後位置 -->
+<xacro:property name="wheel_radius" value="0.0325"/>
+<xacro:property name="wheel_thickness" value="0.025"/>
+<xacro:property name="wheel_distance" value="0.175"/>
+<xacro:property name="wheel_x_offset" value="0.05"/>
 <xacro:property name="body_link_x_dim" value="0.20"/>
 <xacro:property name="body_link_y_dim" value="0.15"/>
@@ -98,5 +96,4 @@
 </joint>
 <link name="base_link"/>
-<!-- 左輪 -->
 <link name="left_wheel">
     <visual>
@@ -104,24 +101,15 @@
             <cylinder radius="${wheel_radius}" length="${wheel_thickness}"/>
         </geometry>
-        <origin xyz="0 0 0" rpy="1.5708 0 0"/>  <!-- link 內設為 0 -->
-        <material name="black">
-            <color rgba="0.1 0.1 0.1 1.0"/>
-        </material>
-    </visual>
-    <collision>
-        <geometry>
-            <cylinder radius="${wheel_radius}" length="${wheel_thickness}"/>
-        </geometry>
-        <origin xyz="0 0 0" rpy="1.5708 0 0"/>  <!-- link 內設為 0 -->
-    </collision>
-    <inertial>
-        <mass value="0.1"/>
-        <origin xyz="0 0 0" rpy="0 0 0"/>
-        <inertia ixx="0.0001" ixy="0.0" ixz="0.0"
-                 iyy="0.0001" iyz="0.0"
-                 izz="0.0001"/>
-    </inertial>
-</link>
-<!-- 右輪 -->
+        <origin xyz="0 0 0" rpy="1.5708 0 0"/>
+        <material name="black"/>
+    </visual>
+    <collision>
+        <geometry>
+            <cylinder radius="${wheel_radius}" length="${wheel_thickness}"/>
+        </geometry>
+        <origin xyz="0 0 0" rpy="1.5708 0 0"/>
+    </collision>
+    <xacro:inertia_wheel/>
+</link>
 <link name="right_wheel">
     <visual>
@@ -129,5 +117,5 @@
             <cylinder radius="${wheel_radius}" length="${wheel_thickness}"/>
         </geometry>
-        <origin xyz="0 0 0" rpy="1.5708 0 0"/>  <!-- link 內設為 0 -->
+        <origin xyz="0 0 0" rpy="1.5708 0 0"/>
         <material name="black"/>
     </visual>
@@ -136,20 +124,12 @@
             <cylinder radius="${wheel_radius}" length="${wheel_thickness}"/>
         </geometry>
-        <origin xyz="0 0 0" rpy="1.5708 0 0"/>  <!-- link 內設為 0 -->
-    </collision>
-    <inertial>
-        <mass value="0.1"/>
-        <origin xyz="0 0 0" rpy="0 0 0"/>
-        <inertia ixx="0.0001" ixy="0.0" ixz="0.0"
-                 iyy="0.0001" iyz="0.0"
-                 izz="0.0001"/>
-    </inertial>
-</link>
-<!-- 輪子關節 - 用你喜歡的格式 -->
+        <origin xyz="0 0 0" rpy="1.5708 0 0"/>
+    </collision>
+    <xacro:inertia_wheel/>
+</link>
 <joint name="left_wheel_joint" type="continuous">
     <parent link="body_link"/>
     <child link="left_wheel"/>
-    <origin xyz="${wheel_x_offset} ${wheel_distance/2} 0" rpy="0 0 0"/>
-    <!-- X=0.05, Y=0.0875, Z=0 -->
+    <origin xyz="${wheel_x_offset} ${wheel_distance/2 + wheel_thickness/2} ${wheel_link_z_location}" rpy="0 0 0"/>
     <axis xyz="0 1 0"/>
 </joint>
@@ -157,8 +137,7 @@
     <parent link="body_link"/>
     <child link="right_wheel"/>
-    <origin xyz="${wheel_x_offset} ${-wheel_distance/2} 0" rpy="0 0 0"/>
-    <!-- X=0.05, Y=-0.0875, Z=0 -->
+    <origin xyz="${wheel_x_offset} ${-wheel_distance/2 - wheel_thickness/2} ${wheel_link_z_location}" rpy="0 0 0"/>
     <axis xyz="0 1 0"/>
-</joint>ㄋ
+</joint>
 <joint name="caster_joint" type="fixed">
     <parent link="body_link"/>

Commit message: model finish

File: install/jetbot_ros/share/jetbot_ros/urdf/jetbot.urdf (robot description, URDF)
Before this commit: robot jetbot, 12 links, 11 joints
Links:
- removed link body_link
- removed link camera_left_link
- removed link camera_mount_link
- removed link camera_pole_link
- removed link camera_right_link
- removed link caster_link
- removed link left_wheel
- removed link right_wheel
- added link arm1, mass 0.0132; collision mesh filename=package://jetbot_ros/meshes/arm1.STL; visual mesh filename=package://jetbot_ros/meshes/arm1.STL
- added link arm2, mass 0.0064; collision mesh filename=package://jetbot_ros/meshes/arm2.STL; visual mesh filename=package://jetbot_ros/meshes/arm2.STL
- added link camera_left, mass 0.00011545; collision mesh filename=package://jetbot_ros/meshes/camera_left.STL; visual mesh filename=package://jetbot_ros/meshes/camera_left.STL
- added link camera_right, mass 0.00011545; collision mesh filename=package://jetbot_ros/meshes/camera_right.STL; visual mesh filename=package://jetbot_ros/meshes/camera_right.STL
- added link caster, mass 0.0080425; collision mesh filename=package://jetbot_ros/meshes/caster.STL; visual mesh filename=package://jetbot_ros/meshes/caster.STL
- added link casterDriver, mass 0.06; collision mesh filename=package://jetbot_ros/meshes/casterDriver.STL; visual mesh filename=package://jetbot_ros/meshes/casterDriver.STL
- added link wheel_left, mass 0.0966027174608247; collision mesh filename=package://jetbot_ros/meshes/wheel_left.STL; visual mesh filename=package://jetbot_ros/meshes/wheel_left.STL
- added link wheel_right, mass 0.0966027174608247; collision mesh filename=package://jetbot_ros/meshes/wheel_right.STL; visual mesh filename=package://jetbot_ros/meshes/wheel_right.STL
- link base_link: mass None -> 0.0768; geometry collision mesh filename=package://jetbot_ros/meshes/base_link.STL; visual mesh filename=package://jetbot_ros/meshes/base_link.STL
Joints:
- removed joint base_link_joint
- removed joint camera_left_joint
- removed joint camera_mount_joint
- removed joint camera_pole_joint
- removed joint camera_right_joint
- removed joint caster_joint
- removed joint left_wheel_joint
- removed joint right_wheel_joint
- added joint arm1: type fixed, parent base_link, child arm1, origin xyz=0.074985 0.00017408 0.055021 rpy=0 0 0
- added joint arm2: type fixed, parent arm1, child arm2, origin xyz=0.0019912 -0.0003142 0.037999 rpy=0 0 0
- added joint cameraLeft: type fixed, parent arm2, child camera_left, origin xyz=0.0023543 0.074021 0.00064658 rpy=0 0 0
- added joint cameraRight: type fixed, parent arm2, child camera_right, origin xyz=0.0036454 -0.073968 -0.00064475 rpy=0 0 0
- added joint caster: type fixed, parent casterDriver, child caster, origin xyz=-0.025083 0.0099121 -0.01492 rpy=-1.5708 0 0
- added joint casterDriver: type fixed, parent base_link, child casterDriver, origin xyz=0.060069 -0.0069739 -0.019048 rpy=0 0 0
- added joint wheelLeft: type continuous, parent base_link, child wheel_left, origin xyz=-0.034751 0.086437 -0.015254 rpy=-1.5708 0 0, axis 0 0 1
- added joint wheelRight: type continuous, parent base_link, child wheel_right, origin xyz=-0.03324 -0.08675 -0.016765 rpy=1.5708 0 0, axis 0 0 1
- joint base_footprint_joint: child body_link -> base_link; origin xyz=0 0 0.0325 rpy=0 0 0 -> xyz=0 0 0.034 rpy=0 0 0
- joint camera_left_optical_joint: origin xyz=0 0 0 rpy=-1.5708 0 -1.5708 -> xyz=0 0 0 rpy=-1.5707963 0 -1.5707963; parent camera_left_link -> camera_left
- joint camera_right_optical_joint: origin xyz=0 0 0 rpy=-1.5708 0 -1.5708 -> xyz=0 0 0 rpy=-1.5707963 0 -1.5707963; parent camera_right_link -> camera_right
